File: bitwise_operator/bitwise_operator_pcb.kicad_pcb (KiCad board)
At the start: 2 copper layers, 121.9 x 149.2 mm, 72 parts, among them J1 Conn_01x03, J2 Conn_02x08_Odd_Even, J3 Conn_02x08_Odd_Even, J4 Conn_02x08_Odd_Even, J5 Conn_02x02_Odd_Even, U1 74LS08, U10 74LS86, U11 74LS86, U12 74LS86, U13 74LS04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

Commit message: part lists
Parts:
- C10: renamed from C5; value 0.5µF -> 0.1µF
Changed lines of the file:
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@@
     (descr "C, Disc series, Radial, pin pitch=5.00mm, , diameter*width=4.3*1.9mm^2, Capacitor, http://www.vishay.com/docs/45233/krseries.pdf")
     (tags "C Disc series Radial pin pitch 5.00mm  diameter 4.3mm width 1.9mm Capacitor")
-    (fp_text reference C5 (at 2.5 -2.2 90) (layer F.SilkS)
+    (fp_text reference C10 (at 2.5 -2.2 90) (layer F.SilkS)
       (effects (font (size 1 1) (thickness 0.15)))
     )
-    (fp_text value 0.5µF (at 2.5 2.2 90) (layer F.Fab)
+    (fp_text value 0.1µF (at 2.5 2.2 90) (layer F.Fab)
       (effects (font (size 1 1) (thickness 0.15)))
     )
