File: bitwise_operator/bus_multiplexer.sch (KiCad schematic (older format))
At the start: 8 parts, among them U16 74LS153, U17 74LS153, U18 74LS153, U19 74LS153, U20 74LS153, U21 74LS153, U22 74LS153, U23 74LS153

Commit message: add bit operations
Parts:
- renumbered U16 to U?, U18 to U?, U20 to U?, U22 to U?, U17 to U?, U19 to U?, U21 to U?, U23 to U?
Changed lines of the file:
@@
 EESchema Schematic File Version 4
+LIBS:computer-cache
 EELAYER 30 0
 EELAYER END
 $Descr A4 11693 8268
 encoding utf-8
-Sheet 7 13
+Sheet 9 29
 Title ""
 Date ""
@@
 $EndDescr
 $Comp
-L 74xx:74LS153 U16
+L 74xx:74LS153 U?
 U 1 1 5F41C685
 P 2350 2250
-F 0 "U16" V 2700 1575 50  0000 L CNN
+F 0 "U?" V 2700 1575 50  0000 L CNN
 F 1 "74LS153" V 2775 1475 50  0000 L CNN
 F 2 "Package_DIP:DIP-16_W7.62mm_LongPads" H 2350 2250 50  0001 C CNN
@@
 	1250 2250 1250 2400
 $Comp
-L power:GND #PWR0111
+L power:GND #PWR?
 U 1 1 5F423E05
 P 1250 2400
-F 0 "#PWR0111" H 1250 2150 50  0001 C CNN
+F 0 "#PWR?" H 1250 2150 50  0001 C CNN
 F 1 "GND" H 1255 2227 50  0000 C CNN
 F 2 "" H 1250 2400 50  0001 C CNN
@@
 	3350 2250 3350 2075
 $Comp
-L power:VCC #PWR0112
+L power:VCC #PWR?
 U 1 1 5F424018
 P 3350 2075
-F 0 "#PWR0112" H 3350 1925 50  0001 C CNN
+F 0 "#PWR?" H 3350 1925 50  0001 C CNN
 F 1 "VCC" H 3367 2248 50  0000 C CNN
 F 2 "" H 3350 2075 50  0001 C CNN
@@
 	3050 775  3050 1750
 $Comp
-L 74xx:74LS153 U18
+L 74xx:74LS153 U?
 U 1 1 5F42F7B7
 P 4500 2250
-F 0 "U18" V 4850 1575 50  0000 L CNN
+F 0 "U?" V 4850 1575 50  0000 L CNN
 F 1 "74LS153" V 4925 1475 50  0000 L CNN
 F 2 "Package_DIP:DIP-16_W7.62mm_LongPads" H 4500 2250 50  0001 C CNN
@@
 	3400 2250 3400 2400
 $Comp
-L power:GND #PWR0113
+L power:GND #PWR?
 U 1 1 5F42F7BE
 P 3400 2400
-F 0 "#PWR0113" H 3400 2150 50  0001 C CNN
+F 0 "#PWR?" H 3400 2150 50  0001 C CNN
 F 1 "GND" H 3405 2227 50  0000 C CNN
 F 2 "" H 3400 2400 50  0001 C CNN
@@
 	5500 2250 5500 2075
 $Comp
-L power:VCC #PWR0114
+L power:VCC #PWR?
 U 1 1 5F42F7C5
 P 5500 2075
-F 0 "#PWR0114" H 5500 1925 50  0001 C CNN
+F 0 "#PWR?" H 5500 1925 50  0001 C CNN
 F 1 "VCC" H 5517 2248 50  0000 C CNN
 F 2 "" H 5500 2075 50  0001 C CNN
@@
 	1650 1425 3800 1425
 $Comp
-L 74xx:74LS153 U20
+L 74xx:74LS153 U?
 U 1 1 5F456CF8
 P 6650 2250
-F 0 "U20" V 7000 1575 50  0000 L CNN
+F 0 "U?" V 7000 1575 50  0000 L CNN
 F 1 "74LS153" V 7075 1475 50  0000 L CNN
 F 2 "Package_DIP:DIP-16_W7.62mm_LongPads" H 6650 2250 50  0001 C CNN
@@
 	5550 2250 5550 2400
 $Comp
-L power:GND #PWR0115
+L power:GND #PWR?
 U 1 1 5F456CFF
 P 5550 2400
-F 0 "#PWR0115" H 5550 2150 50  0001 C CNN
+F 0 "#PWR?" H 5550 2150 50  0001 C CNN
 F 1 "GND" H 5555 2227 50  0000 C CNN
 F 2 "" H 5550 2400 50  0001 C CNN
@@
 	7650 2250 7650 2075
 $Comp
-L power:VCC #PWR0116
+L power:VCC #PWR?
 U 1 1 5F456D06
 P 7650 2075
-F 0 "#PWR0116" H 7650 1925 50  0001 C CNN
+F 0 "#PWR?" H 7650 1925 50  0001 C CNN
 F 1 "VCC" H 7667 2248 50  0000 C CNN
 F 2 "" H 7650 2075 50  0001 C CNN
@@
 	7350 775  7350 1750
 $Comp
-L 74xx:74LS153 U22
+L 74xx:74LS153 U?
 U 1 1 5F456D38
 P 8800 2250
-F 0 "U22" V 9150 1575 50  0000 L CNN
+F 0 "U?" V 9150 1575 50  0000 L CNN
 F 1 "74LS153" V 9225 1475 50  0000 L CNN
 F 2 "Package_DIP:DIP-16_W7.62mm_LongPads" H 8800 2250 50  0001 C CNN
@@
 	7700 2250 7700 2400
 $Comp
-L power:GND #PWR0117
+L power:GND #PWR?
 U 1 1 5F456D3F
 P 7700 2400
-F 0 "#PWR0117" H 7700 2150 50  0001 C CNN
+F 0 "#PWR?" H 7700 2150 50  0001 C CNN
 F 1 "GND" H 7705 2227 50  0000 C CNN
 F 2 "" H 7700 2400 50  0001 C CNN
@@
 	9800 2250 9800 2075
 $Comp
-L power:VCC #PWR0118
+L power:VCC #PWR?
 U 1 1 5F456D46
 P 9800 2075
-F 0 "#PWR0118" H 9800 1925 50  0001 C CNN
+F 0 "#PWR?" H 9800 1925 50  0001 C CNN
 F 1 "VCC" H 9817 2248 50  0000 C CNN
 F 2 "" H 9800 2075 50  0001 C CNN
@@
 	3800 1425 5950 1425
 $Comp
-L 74xx:74LS153 U17
+L 74xx:74LS153 U?
 U 1 1 5F47E1F4
 P 2350 4050
-F 0 "U17" V 2700 3375 50  0000 L CNN
+F 0 "U?" V 2700 3375 50  0000 L CNN
 F 1 "74LS153" V 2775 3275 50  0000 L CNN
 F 2 "Package_DIP:DIP-16_W7.62mm_LongPads" H 2350 4050 50  0001 C CNN
@@
 	1250 4050 1250 3900
 $Comp
-L power:GND #PWR0119
+L power:GND #PWR?
 U 1 1 5F47E1FB
 P 1250 3900
-F 0 "#PWR0119" H 1250 3650 50  0001 C CNN
+F 0 "#PWR?" H 1250 3650 50  0001 C CNN
 F 1 "GND" H 1255 3727 50  0000 C CNN
 F 2 "" H 1250 3900 50  0001 C CNN
@@
 	3350 4050 3350 4225
 $Comp
-L power:VCC #PWR0120
+L power:VCC #PWR?
 U 1 1 5F47E202
 P 3350 4225
-F 0 "#PWR0120" H 3350 4075 50  0001 C CNN
+F 0 "#PWR?" H 3350 4075 50  0001 C CNN
 F 1 "VCC" H 3367 4398 50  0000 C CNN
 F 2 "" H 3350 4225 50  0001 C CNN
@@
 	3050 5525 3050 4550
 $Comp
-L 74xx:74LS153 U19
+L 74xx:74LS153 U?
 U 1 1 5F47E234
 P 4500 4050
-F 0 "U19" V 4850 3375 50  0000 L CNN
+F 0 "U?" V 4850 3375 50  0000 L CNN
 F 1 "74LS153" V 4925 3275 50  0000 L CNN
 F 2 "Package_DIP:DIP-16_W7.62mm_LongPads" H 4500 4050 50  0001 C CNN
@@
 	3400 4050 3400 3900
 $Comp
-L power:GND #PWR0121
+L power:GND #PWR?
 U 1 1 5F47E23B
 P 3400 3900
-F 0 "#PWR0121" H 3400 3650 50  0001 C CNN
+F 0 "#PWR?" H 3400 3650 50  0001 C CNN
 F 1 "GND" H 3405 3727 50  0000 C CNN
 F 2 "" H 3400 3900 50  0001 C CNN
@@
 	5500 4050 5500 4225
 $Comp
-L power:VCC #PWR0122
+L power:VCC #PWR?
 U 1 1 5F47E242
 P 5500 4225
-F 0 "#PWR0122" H 5500 4075 50  0001 C CNN
+F 0 "#PWR?" H 5500 4075 50  0001 C CNN
 F 1 "VCC" H 5517 4398 50  0000 C CNN
 F 2 "" H 5500 4225 50  0001 C CNN
@@
 	1650 4875 3800 4875
 $Comp
-L 74xx:74LS153 U21
+L 74xx:74LS153 U?
 U 1 1 5F47E274
 P 6650 4050
-F 0 "U21" V 7000 3375 50  0000 L CNN
+F 0 "U?" V 7000 3375 50  0000 L CNN
 F 1 "74LS153" V 7075 3275 50  0000 L CNN
 F 2 "Package_DIP:DIP-16_W7.62mm_LongPads" H 6650 4050 50  0001 C CNN
@@
 	5550 4050 5550 3900
 $Comp
-L power:GND #PWR0123
+L power:GND #PWR?
 U 1 1 5F47E27B
 P 5550 3900
-F 0 "#PWR0123" H 5550 3650 50  0001 C CNN
+F 0 "#PWR?" H 5550 3650 50  0001 C CNN
 F 1 "GND" H 5555 3727 50  0000 C CNN
 F 2 "" H 5550 3900 50  0001 C CNN
@@
 	7650 4050 7650 4225
 $Comp
-L power:VCC #PWR0124
+L power:VCC #PWR?
 U 1 1 5F47E282
 P 7650 4225
-F 0 "#PWR0124" H 7650 4075 50  0001 C CNN
+F 0 "#PWR?" H 7650 4075 50  0001 C CNN
 F 1 "VCC" H 7667 4398 50  0000 C CNN
 F 2 "" H 7650 4225 50  0001 C CNN
@@
 	7350 5525 7350 4550
 $Comp
-L 74xx:74LS153 U23
+L 74xx:74LS153 U?
 U 1 1 5F47E2B1
 P 8800 4050
-F 0 "U23" V 9150 3375 50  0000 L CNN
+F 0 "U?" V 9150 3375 50  0000 L CNN
 F 1 "74LS153" V 9225 3275 50  0000 L CNN
 F 2 "Package_DIP:DIP-16_W7.62mm_LongPads" H 8800 4050 50  0001 C CNN
@@
 	7700 4050 7700 3900
 $Comp
-L power:GND #PWR0125
+L power:GND #PWR?
 U 1 1 5F47E2B8
 P 7700 3900
-F 0 "#PWR0125" H 7700 3650 50  0001 C CNN
+F 0 "#PWR?" H 7700 3650 50  0001 C CNN
 F 1 "GND" H 7705 3727 50  0000 C CNN
 F 2 "" H 7700 3900 50  0001 C CNN
@@
 	9800 4050 9800 4225
 $Comp
-L power:VCC #PWR0126
+L power:VCC #PWR?
 U 1 1 5F47E2BF
 P 9800 4225
-F 0 "#PWR0126" H 9800 4075 50  0001 C CNN
+F 0 "#PWR?" H 9800 4075 50  0001 C CNN
 F 1 "VCC" H 9817 4398 50  0000 C CNN
 F 2 "" H 9800 4225 50  0001 C CNN
@@
 	8100 4875 10150 4875
 $Comp
-L power:GND #PWR0127
+L power:GND #PWR?
 U 1 1 5F4D5348
 P 1200 1650
-F 0 "#PWR0127" H 1200 1400 50  0001 C CNN
+F 0 "#PWR?" H 1200 1400 50  0001 C CNN
 F 1 "GND" V 1205 1522 50  0000 R CNN
 F 2 "" H 1200 1650 50  0001 C CNN

Commit message: part lists
Parts:
- gave numbers to parts that had none: 8
Changed lines of the file:
@@
 EESchema Schematic File Version 4
-LIBS:computer-cache
+LIBS:bitwise_operator_pcb-cache
 EELAYER 30 0
 EELAYER END
 $Descr A4 11693 8268
 encoding utf-8
-Sheet 9 36
+Sheet 9 13
 Title ""
 Date ""
@@
 $EndDescr
 $Comp
-L 74xx:74LS153 U?
+L 74xx:74LS153 U16
 U 1 1 5F41C685
 P 2350 2250
-F 0 "U?" V 2700 1575 50  0000 L CNN
+F 0 "U16" V 2700 1575 50  0000 L CNN
 F 1 "74LS153" V 2775 1475 50  0000 L CNN
 F 2 "Package_DIP:DIP-16_W7.62mm_LongPads" H 2350 2250 50  0001 C CNN
@@
 	1250 2250 1250 2400
 $Comp
-L power:GND #PWR?
+L power:GND #PWR04
 U 1 1 5F423E05
 P 1250 2400
-F 0 "#PWR?" H 1250 2150 50  0001 C CNN
+F 0 "#PWR04" H 1250 2150 50  0001 C CNN
 F 1 "GND" H 1255 2227 50  0000 C CNN
 F 2 "" H 1250 2400 50  0001 C CNN
@@
 	3350 2250 3350 2075
 $Comp
-L power:VCC #PWR?
+L power:VCC #PWR06
 U 1 1 5F424018
 P 3350 2075
-F 0 "#PWR?" H 3350 1925 50  0001 C CNN
+F 0 "#PWR06" H 3350 1925 50  0001 C CNN
 F 1 "VCC" H 3367 2248 50  0000 C CNN
 F 2 "" H 3350 2075 50  0001 C CNN
@@
 	3050 775  3050 1750
 $Comp
-L 74xx:74LS153 U?
+L 74xx:74LS153 U18
 U 1 1 5F42F7B7
 P 4500 2250
-F 0 "U?" V 4850 1575 50  0000 L CNN
+F 0 "U18" V 4850 1575 50  0000 L CNN
 F 1 "74LS153" V 4925 1475 50  0000 L CNN
 F 2 "Package_DIP:DIP-16_W7.62mm_LongPads" H 4500 2250 50  0001 C CNN
@@
 	3400 2250 3400 2400
 $Comp
-L power:GND #PWR?
+L power:GND #PWR08
 U 1 1 5F42F7BE
 P 3400 2400
-F 0 "#PWR?" H 3400 2150 50  0001 C CNN
+F 0 "#PWR08" H 3400 2150 50  0001 C CNN
 F 1 "GND" H 3405 2227 50  0000 C CNN
 F 2 "" H 3400 2400 50  0001 C CNN
@@
 	5500 2250 5500 2075
 $Comp
-L power:VCC #PWR?
+L power:VCC #PWR010
 U 1 1 5F42F7C5
 P 5500 2075
-F 0 "#PWR?" H 5500 1925 50  0001 C CNN
+F 0 "#PWR010" H 5500 1925 50  0001 C CNN
 F 1 "VCC" H 5517 2248 50  0000 C CNN
 F 2 "" H 5500 2075 50  0001 C CNN
@@
 	1650 1425 3800 1425
 $Comp
-L 74xx:74LS153 U?
+L 74xx:74LS153 U20
 U 1 1 5F456CF8
 P 6650 2250
-F 0 "U?" V 7000 1575 50  0000 L CNN
+F 0 "U20" V 7000 1575 50  0000 L CNN
 F 1 "74LS153" V 7075 1475 50  0000 L CNN
 F 2 "Package_DIP:DIP-16_W7.62mm_LongPads" H 6650 2250 50  0001 C CNN
@@
 	5550 2250 5550 2400
 $Comp
-L power:GND #PWR?
+L power:GND #PWR012
 U 1 1 5F456CFF
 P 5550 2400
-F 0 "#PWR?" H 5550 2150 50  0001 C CNN
+F 0 "#PWR012" H 5550 2150 50  0001 C CNN
 F 1 "GND" H 5555 2227 50  0000 C CNN
 F 2 "" H 5550 2400 50  0001 C CNN
@@
 	7650 2250 7650 2075
 $Comp
-L power:VCC #PWR?
+L power:VCC #PWR014
 U 1 1 5F456D06
 P 7650 2075
-F 0 "#PWR?" H 7650 1925 50  0001 C CNN
+F 0 "#PWR014" H 7650 1925 50  0001 C CNN
 F 1 "VCC" H 7667 2248 50  0000 C CNN
 F 2 "" H 7650 2075 50  0001 C CNN
@@
 	7350 775  7350 1750
 $Comp
-L 74xx:74LS153 U?
+L 74xx:74LS153 U22
 U 1 1 5F456D38
 P 8800 2250
-F 0 "U?" V 9150 1575 50  0000 L CNN
+F 0 "U22" V 9150 1575 50  0000 L CNN
 F 1 "74LS153" V 9225 1475 50  0000 L CNN
 F 2 "Package_DIP:DIP-16_W7.62mm_LongPads" H 8800 2250 50  0001 C CNN
@@
 	7700 2250 7700 2400
 $Comp
-L power:GND #PWR?
+L power:GND #PWR016
 U 1 1 5F456D3F
 P 7700 2400
-F 0 "#PWR?" H 7700 2150 50  0001 C CNN
+F 0 "#PWR016" H 7700 2150 50  0001 C CNN
 F 1 "GND" H 7705 2227 50  0000 C CNN
 F 2 "" H 7700 2400 50  0001 C CNN
@@
 	9800 2250 9800 2075
 $Comp
-L power:VCC #PWR?
+L power:VCC #PWR018
 U 1 1 5F456D46
 P 9800 2075
-F 0 "#PWR?" H 9800 1925 50  0001 C CNN
+F 0 "#PWR018" H 9800 1925 50  0001 C CNN
 F 1 "VCC" H 9817 2248 50  0000 C CNN
 F 2 "" H 9800 2075 50  0001 C CNN
@@
 	3800 1425 5950 1425
 $Comp
-L 74xx:74LS153 U?
+L 74xx:74LS153 U17
 U 1 1 5F47E1F4
 P 2350 4050
-F 0 "U?" V 2700 3375 50  0000 L CNN
+F 0 "U17" V 2700 3375 50  0000 L CNN
 F 1 "74LS153" V 2775 3275 50  0000 L CNN
 F 2 "Package_DIP:DIP-16_W7.62mm_LongPads" H 2350 4050 50  0001 C CNN
@@
 	1250 4050 1250 3900
 $Comp
-L power:GND #PWR?
+L power:GND #PWR05
 U 1 1 5F47E1FB
 P 1250 3900
-F 0 "#PWR?" H 1250 3650 50  0001 C CNN
+F 0 "#PWR05" H 1250 3650 50  0001 C CNN
 F 1 "GND" H 1255 3727 50  0000 C CNN
 F 2 "" H 1250 3900 50  0001 C CNN
@@
 	3350 4050 3350 4225
 $Comp
-L power:VCC #PWR?
+L power:VCC #PWR07
 U 1 1 5F47E202
 P 3350 4225
-F 0 "#PWR?" H 3350 4075 50  0001 C CNN
+F 0 "#PWR07" H 3350 4075 50  0001 C CNN
 F 1 "VCC" H 3367 4398 50  0000 C CNN
 F 2 "" H 3350 4225 50  0001 C CNN
@@
 	3050 5525 3050 4550
 $Comp
-L 74xx:74LS153 U?
+L 74xx:74LS153 U19
 U 1 1 5F47E234
 P 4500 4050
-F 0 "U?" V 4850 3375 50  0000 L CNN
+F 0 "U19" V 4850 3375 50  0000 L CNN
 F 1 "74LS153" V 4925 3275 50  0000 L CNN
 F 2 "Package_DIP:DIP-16_W7.62mm_LongPads" H 4500 4050 50  0001 C CNN
@@
 	3400 4050 3400 3900
 $Comp
-L power:GND #PWR?
+L power:GND #PWR09
 U 1 1 5F47E23B
 P 3400 3900
-F 0 "#PWR?" H 3400 3650 50  0001 C CNN
+F 0 "#PWR09" H 3400 3650 50  0001 C CNN
 F 1 "GND" H 3405 3727 50  0000 C CNN
 F 2 "" H 3400 3900 50  0001 C CNN
@@
 	5500 4050 5500 4225
 $Comp
-L power:VCC #PWR?
+L power:VCC #PWR011
 U 1 1 5F47E242
 P 5500 4225
-F 0 "#PWR?" H 5500 4075 50  0001 C CNN
+F 0 "#PWR011" H 5500 4075 50  0001 C CNN
 F 1 "VCC" H 5517 4398 50  0000 C CNN
 F 2 "" H 5500 4225 50  0001 C CNN
@@
 	1650 4875 3800 4875
 $Comp
-L 74xx:74LS153 U?
+L 74xx:74LS153 U21
 U 1 1 5F47E274
 P 6650 4050
-F 0 "U?" V 7000 3375 50  0000 L CNN
+F 0 "U21" V 7000 3375 50  0000 L CNN
 F 1 "74LS153" V 7075 3275 50  0000 L CNN
 F 2 "Package_DIP:DIP-16_W7.62mm_LongPads" H 6650 4050 50  0001 C CNN
@@
 	5550 4050 5550 3900
 $Comp
-L power:GND #PWR?
+L power:GND #PWR013
 U 1 1 5F47E27B
 P 5550 3900
-F 0 "#PWR?" H 5550 3650 50  0001 C CNN
+F 0 "#PWR013" H 5550 3650 50  0001 C CNN
 F 1 "GND" H 5555 3727 50  0000 C CNN
 F 2 "" H 5550 3900 50  0001 C CNN
@@
 	7650 4050 7650 4225
 $Comp
-L power:VCC #PWR?
+L power:VCC #PWR015
 U 1 1 5F47E282
 P 7650 4225
-F 0 "#PWR?" H 7650 4075 50  0001 C CNN
+F 0 "#PWR015" H 7650 4075 50  0001 C CNN
 F 1 "VCC" H 7667 4398 50  0000 C CNN
 F 2 "" H 7650 4225 50  0001 C CNN
@@
 	7350 5525 7350 4550
 $Comp
-L 74xx:74LS153 U?
+L 74xx:74LS153 U23
 U 1 1 5F47E2B1
 P 8800 4050
-F 0 "U?" V 9150 3375 50  0000 L CNN
+F 0 "U23" V 9150 3375 50  0000 L CNN
 F 1 "74LS153" V 9225 3275 50  0000 L CNN
 F 2 "Package_DIP:DIP-16_W7.62mm_LongPads" H 8800 4050 50  0001 C CNN
@@
 	7700 4050 7700 3900
 $Comp
-L power:GND #PWR?
+L power:GND #PWR017
 U 1 1 5F47E2B8
 P 7700 3900
-F 0 "#PWR?" H 7700 3650 50  0001 C CNN
+F 0 "#PWR017" H 7700 3650 50  0001 C CNN
 F 1 "GND" H 7705 3727 50  0000 C CNN
 F 2 "" H 7700 3900 50  0001 C CNN
@@
 	9800 4050 9800 4225
 $Comp
-L power:VCC #PWR?
+L power:VCC #PWR019
 U 1 1 5F47E2BF
 P 9800 4225
-F 0 "#PWR?" H 9800 4075 50  0001 C CNN
+F 0 "#PWR019" H 9800 4075 50  0001 C CNN
 F 1 "VCC" H 9817 4398 50  0000 C CNN
 F 2 "" H 9800 4225 50  0001 C CNN
@@
 	8100 4875 10150 4875
 $Comp
-L power:GND #PWR?
+L power:GND #PWR03
 U 1 1 5F4D5348
 P 1200 1650
-F 0 "#PWR?" H 1200 1400 50  0001 C CNN
+F 0 "#PWR03" H 1200 1400 50  0001 C CNN
 F 1 "GND" V 1205 1522 50  0000 R CNN
 F 2 "" H 1200 1650 50  0001 C CNN
