File: buttons/buttons_pcb.kicad_pcb (KiCad board)
At the start: 2 copper layers, 93.2 x 50.1 mm, 30 parts, among them J1 Conn_01x02, J2 Conn_02x02_Odd_Even, J3 Conn_02x08_Odd_Even, SW1 SW_Push, SW2 SW_Push, SW3 SW_Push, SW4 SW_Push, SW5 SW_Push, U1 74LS04, U2 74LS375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

Commit message: part lists
Parts:
- renumbered U4 to U24, U5 to U25
Changed lines of the file:
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@@
     (solder_mask_min_width 0.25)
     (aux_axis_origin 0 0)
-    (visible_elements FFFFFF7F)
+    (visible_elements 7FFFFFFF)
     (pcbplotparams
       (layerselection 0x010fc_ffffffff)
@@
     (descr "20-lead though-hole mounted DIP package, row spacing 7.62 mm (300 mils), LongPads")
     (tags "THT DIP DIL PDIP 2.54mm 7.62mm 300mil LongPads")
-    (fp_text reference U5 (at 3.81 -2.33 90) (layer F.SilkS)
+    (fp_text reference U25 (at 3.81 -2.33 90) (layer F.SilkS)
       (effects (font (size 1 1) (thickness 0.15)))
     )
@@
     (descr "20-lead though-hole mounted DIP package, row spacing 7.62 mm (300 mils), LongPads")
     (tags "THT DIP DIL PDIP 2.54mm 7.62mm 300mil LongPads")
-    (fp_text reference U4 (at 3.81 -2.33 90) (layer F.SilkS)
-      (effects (font (size 1 1) (thickness 0.15)))
-    )
+    (fp_text reference U24 (at 3.81 -2.33 90) (layer F.SilkS)
+      (effects (font (size 1 1) (thickness 0.15)))
+    )
