File: control_unit/control_unit_pcb.kicad_pcb (KiCad board)
At the start: 2 copper layers, 252.7 x 133.2 mm, 195 parts, among them J1 Conn_01x04, J10 Conn_01x08, J11 Conn_01x08, J12 Conn_01x08, J13 Conn_01x08, J2 Conn_01x08, J3 Conn_01x08, J4 Conn_01x03, J5 Conn_02x04_Odd_Even, J6 Conn_02x04_Odd_Even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

Commit message: part lists
Parts:
- renumbered U10 to U24, U11 to U25
Changed lines of the file:
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@@
     (descr "20-lead though-hole mounted DIP package, row spacing 7.62 mm (300 mils), LongPads")
     (tags "THT DIP DIL PDIP 2.54mm 7.62mm 300mil LongPads")
-    (fp_text reference U11 (at 3.81 -2.33) (layer F.SilkS)
+    (fp_text reference U25 (at 3.81 -2.33) (layer F.SilkS)
       (effects (font (size 1 1) (thickness 0.15)))
     )
@@
     (descr "20-lead though-hole mounted DIP package, row spacing 7.62 mm (300 mils), LongPads")
     (tags "THT DIP DIL PDIP 2.54mm 7.62mm 300mil LongPads")
-    (fp_text reference U10 (at 3.81 -2.33) (layer F.SilkS)
+    (fp_text reference U24 (at 3.81 -2.33) (layer F.SilkS)
       (effects (font (size 1 1) (thickness 0.15)))
     )
