File: display/display_pcb.kicad_pcb (KiCad board)
At the start: 2 copper layers, 21 parts, among them IC1 CD40109BE, IC2 CD40109BE, IC3 CD40109BE, IC4 CD40109BE, J1 Conn_02x03_Odd_Even, J2 Conn_02x08_Odd_Even, J3 Conn_02x02_Odd_Even, U1 LP2950-3.0_TO92, U2 74LS244

Commit message: part lists
Parts:
- renumbered C9 to C1, C5 to C2, C1 to C4, C4 to C5, C2 to C6, C8 to C7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
