File: program_counter/program_counter_pcb.kicad_pcb (KiCad board)
At the start: 2 copper layers, 116.8 x 46.9 mm, 45 parts, among them J1 Conn_01x04, J2 Conn_02x02_Odd_Even, J3 Conn_02x08_Odd_Even, U1 74LS163, U2 74LS163, U3 74LS163, U4 74LS163, U5 74LS244, U6 74LS244

Commit message: part lists
Parts:
- renumbered U5 to U24, U6 to U25
Changed lines of the file:
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@@
     (descr "20-lead though-hole mounted DIP package, row spacing 7.62 mm (300 mils), LongPads")
     (tags "THT DIP DIL PDIP 2.54mm 7.62mm 300mil LongPads")
-    (fp_text reference U6 (at 3.81 -2.33 90) (layer F.SilkS)
+    (fp_text reference U25 (at 3.81 -2.33 90) (layer F.SilkS)
       (effects (font (size 1 1) (thickness 0.15)))
     )
@@
     (descr "20-lead though-hole mounted DIP package, row spacing 7.62 mm (300 mils), LongPads")
     (tags "THT DIP DIL PDIP 2.54mm 7.62mm 300mil LongPads")
-    (fp_text reference U5 (at 3.81 -2.33 90) (layer F.SilkS)
+    (fp_text reference U24 (at 3.81 -2.33 90) (layer F.SilkS)
       (effects (font (size 1 1) (thickness 0.15)))
     )
