File: program_counter/program_counter.sch (KiCad schematic (older format))
At the start: 8 parts

Commit message: part lists
Parts:
- gave numbers to parts that had none: 8
Changed lines of the file:
@@
 EESchema Schematic File Version 4
-LIBS:computer-cache
+LIBS:program_counter_pcb-cache
 EELAYER 30 0
 EELAYER END
 $Descr A4 11693 8268
 encoding utf-8
-Sheet 4 36
+Sheet 4 6
 Title ""
 Date ""
@@
 BUS[0..15]
 $Comp
-L 74xx:74LS163 U?
+L 74xx:74LS163 U1
 U 1 1 5EE683D1
 P 3475 3175
-F 0 "U?" H 3475 4156 50  0000 C CNN
+F 0 "U1" H 3475 4156 50  0000 C CNN
 F 1 "74LS163" H 3475 4065 50  0000 C CNN
 F 2 "Package_DIP:DIP-16_W7.62mm_LongPads" H 3475 3175 50  0001 C CNN
@@
 $EndComp
 $Comp
-L 74xx:74LS163 U?
+L 74xx:74LS163 U2
 U 1 1 5EE6C173
 P 5425 3175
-F 0 "U?" H 5425 4156 50  0000 C CNN
+F 0 "U2" H 5425 4156 50  0000 C CNN
 F 1 "74LS163" H 5425 4065 50  0000 C CNN
 F 2 "Package_DIP:DIP-16_W7.62mm_LongPads" H 5425 3175 50  0001 C CNN
@@
 $EndComp
 $Comp
-L 74xx:74LS163 U?
+L 74xx:74LS163 U3
 U 1 1 5EE6F0B9
 P 7375 3175
-F 0 "U?" H 7375 4156 50  0000 C CNN
+F 0 "U3" H 7375 4156 50  0000 C CNN
 F 1 "74LS163" H 7375 4065 50  0000 C CNN
 F 2 "Package_DIP:DIP-16_W7.62mm_LongPads" H 7375 3175 50  0001 C CNN
@@
 	3375 2150 5325 2150
 $Comp
-L power:VCC #PWR?
+L power:VCC #PWR013
 U 1 1 5EEA271D
 P 9125 2575
-F 0 "#PWR?" H 9125 2425 50  0001 C CNN
+F 0 "#PWR013" H 9125 2425 50  0001 C CNN
 F 1 "VCC" H 9142 2748 50  0000 C CNN
 F 2 "" H 9125 2575 50  0001 C CNN
@@
 	9125 2575 9125 2675
 $Comp
-L power:VCC #PWR?
+L power:VCC #PWR014
 U 1 1 5EEA462B
 P 10125 2975
-F 0 "#PWR?" H 10125 2825 50  0001 C CNN
+F 0 "#PWR014" H 10125 2825 50  0001 C CNN
 F 1 "VCC" H 10142 3148 50  0000 C CNN
 F 2 "" H 10125 2975 50  0001 C CNN
@@
 	10125 3175 10125 2975
 $Comp
-L 74xx:74LS163 U?
+L 74xx:74LS163 U4
 U 1 1 5EE6F0BF
 P 9325 3175
-F 0 "U?" H 9325 4156 50  0000 C CNN
+F 0 "U4" H 9325 4156 50  0000 C CNN
 F 1 "74LS163" H 9325 4065 50  0000 C CNN
 F 2 "Package_DIP:DIP-16_W7.62mm_LongPads" H 9325 3175 50  0001 C CNN
@@
 $EndComp
 $Comp
-L power:VCC #PWR?
+L power:VCC #PWR011
 U 1 1 5EEA823B
 P 8175 2975
-F 0 "#PWR?" H 8175 2825 50  0001 C CNN
+F 0 "#PWR011" H 8175 2825 50  0001 C CNN
 F 1 "VCC" H 8192 3148 50  0000 C CNN
 F 2 "" H 8175 2975 50  0001 C CNN
@@
 	8175 3175 8175 2975
 $Comp
-L power:VCC #PWR?
+L power:VCC #PWR09
 U 1 1 5EEA9CD5
 P 6225 2975
-F 0 "#PWR?" H 6225 2825 50  0001 C CNN
+F 0 "#PWR09" H 6225 2825 50  0001 C CNN
 F 1 "VCC" H 6242 3148 50  0000 C CNN
 F 2 "" H 6225 2975 50  0001 C CNN
@@
 	6225 3175 6225 2975
 $Comp
-L power:VCC #PWR?
+L power:VCC #PWR07
 U 1 1 5EEAB8E7
 P 4275 2975
-F 0 "#PWR?" H 4275 2825 50  0001 C CNN
+F 0 "#PWR07" H 4275 2825 50  0001 C CNN
 F 1 "VCC" H 4292 3148 50  0000 C CNN
 F 2 "" H 4275 2975 50  0001 C CNN
@@
 	2675 3175 2675 3375
 $Comp
-L power:GND #PWR?
+L power:GND #PWR05
 U 1 1 5EEAF398
 P 2675 3375
-F 0 "#PWR?" H 2675 3125 50  0001 C CNN
+F 0 "#PWR05" H 2675 3125 50  0001 C CNN
 F 1 "GND" H 2680 3202 50  0000 C CNN
 F 2 "" H 2675 3375 50  0001 C CNN
@@
 	4625 3175 4625 3375
 $Comp
-L power:GND #PWR?
+L power:GND #PWR08
 U 1 1 5EEB1876
 P 4625 3375
-F 0 "#PWR?" H 4625 3125 50  0001 C CNN
+F 0 "#PWR08" H 4625 3125 50  0001 C CNN
 F 1 "GND" H 4630 3202 50  0000 C CNN
 F 2 "" H 4625 3375 50  0001 C CNN
@@
 	6575 3175 6575 3375
 $Comp
-L power:GND #PWR?
+L power:GND #PWR010
 U 1 1 5EEB3741
 P 6575 3375
-F 0 "#PWR?" H 6575 3125 50  0001 C CNN
+F 0 "#PWR010" H 6575 3125 50  0001 C CNN
 F 1 "GND" H 6580 3202 50  0000 C CNN
 F 2 "" H 6575 3375 50  0001 C CNN
@@
 	8525 3175 8525 3375
 $Comp
-L power:GND #PWR?
+L power:GND #PWR012
 U 1 1 5EEB55B1
 P 8525 3375
-F 0 "#PWR?" H 8525 3125 50  0001 C CNN
+F 0 "#PWR012" H 8525 3125 50  0001 C CNN
 F 1 "GND" H 8530 3202 50  0000 C CNN
 F 2 "" H 8525 3375 50  0001 C CNN
@@
 NoConn ~ 3475 3675
 $Comp
-L Device:C C?
+L Device:C C1
 U 1 1 5EF1A1A3
 P 2525 5300
-F 0 "C?" V 2273 5300 50  0000 C CNN
+F 0 "C1" V 2273 5300 50  0000 C CNN
 F 1 "0.1µF" V 2364 5300 50  0000 C CNN
 F 2 "Capacitor_THT:C_Disc_D4.3mm_W1.9mm_P5.00mm" H 2563 5150 50  0001 C CNN
@@
 $EndComp
 $Comp
-L Device:C C?
+L Device:C C2
 U 1 1 5EF1A6C4
 P 2525 5700
-F 0 "C?" V 2273 5700 50  0000 C CNN
+F 0 "C2" V 2273 5700 50  0000 C CNN
 F 1 "0.1µF" V 2364 5700 50  0000 C CNN
 F 2 "Capacitor_THT:C_Disc_D4.3mm_W1.9mm_P5.00mm" H 2563 5550 50  0001 C CNN
@@
 $EndComp
 $Comp
-L Device:C C?
+L Device:C C3
 U 1 1 5EF1D830
 P 2525 6100
-F 0 "C?" V 2273 6100 50  0000 C CNN
+F 0 "C3" V 2273 6100 50  0000 C CNN
 F 1 "0.1µF" V 2364 6100 50  0000 C CNN
 F 2 "Capacitor_THT:C_Disc_D4.3mm_W1.9mm_P5.00mm" H 2563 5950 50  0001 C CNN
@@
 	2250 5700 2375 5700
 $Comp
-L power:VCC #PWR?
+L power:VCC #PWR04
 U 1 1 5EF359E4
 P 2250 5700
-F 0 "#PWR?" H 2250 5550 50  0001 C CNN
+F 0 "#PWR04" H 2250 5550 50  0001 C CNN
 F 1 "VCC" V 2268 5827 50  0000 L CNN
 F 2 "" H 2250 5700 50  0001 C CNN
@@
 $EndComp
 $Comp
-L power:GND #PWR?
+L power:GND #PWR06
 U 1 1 5EF396BA
 P 2800 5700
-F 0 "#PWR?" H 2800 5450 50  0001 C CNN
+F 0 "#PWR06" H 2800 5450 50  0001 C CNN
 F 1 "GND" V 2805 5572 50  0000 R CNN
 F 2 "" H 2800 5700 50  0001 C CNN
@@
 	2800 5700 2675 5700
 $Comp
-L power:VCC #PWR?
+L power:VCC #PWR03
 U 1 1 5EF40605
 P 2150 2875
-F 0 "#PWR?" H 2150 2725 50  0001 C CNN
+F 0 "#PWR03" H 2150 2725 50  0001 C CNN
 F 1 "VCC" H 2168 3048 50  0000 C CNN
 F 2 "" H 2150 2875 50  0001 C CNN
@@
 $EndComp
 $Comp
-L Device:R R?
+L Device:R R16
 U 1 1 5EF411BB
 P 2150 2575
-F 0 "R?" H 2220 2621 50  0000 L CNN
+F 0 "R16" H 2220 2621 50  0000 L CNN
 F 1 "50K" H 2220 2530 50  0000 L CNN
 F 2 "Resistor_THT:R_Axial_DIN0207_L6.3mm_D2.5mm_P7.62mm_Horizontal" V 2080 2575 50  0001 C CNN
