File: clock.sch (KiCad schematic (older format))
At the start: 35 parts

Commit message: Commit uncomitted changes. no clue what I had done last time
Other:
- note added: "TODO update with actual circuit"
Changed lines of the file:
@@
 Text HLabel 4800 5150 0    50   Input ~ 0
 HLT_CLK
+Text Notes 5125 3225 0    50   ~ 0
+TODO update with actual circuit
 $EndSCHEMATC
